Commit message: customRobotBasicStack: updated the description with 2 caster wheels

File: amr_description/urdf/amr.xacro (robot description, xacro)
@@ -32,6 +32,6 @@
     </visual>
     <!-- caster front -->
-    <collision name="caster_front_collision">
-      <origin rpy=" 0 0 0" xyz="0.3 0 -0.05"/>
+    <collision name="caster_left_collision">
+      <origin rpy=" 0 0 0" xyz="0.3 0.14 -0.025"/>
       <geometry>
         <sphere radius="0.05"/>
@@ -48,6 +48,28 @@
       </surface>
     </collision>
-    <visual name="caster_front_visual">
-      <origin rpy=" 0 0 0" xyz="0.15 0 -0.05"/>
+    <visual name="caster_left_visual">
+      <origin rpy=" 0 0 0" xyz="0.15 0.07 -0.05"/>
+      <geometry>
+        <sphere radius="0.05"/>
+      </geometry>
+    </visual>
+    <collision name="caster_right_collision">
+      <origin rpy=" 0 0 0" xyz="0.3 0.14 -0.05"/>
+      <geometry>
+        <sphere radius="0.05"/>
+      </geometry>
+      <surface>
+        <friction>
+          <ode>
+            <mu>0</mu>
+            <mu2>0</mu2>
+            <slip1>1.0</slip1>
+            <slip2>1.0</slip2>
+          </ode>
+        </friction>
+      </surface>
+    </collision>
+    <visual name="caster_right_visual">
+      <origin rpy=" 0 0 0" xyz="0.15 -0.07 -0.05"/>
       <geometry>
         <sphere radius="0.05"/>
